File: hardware/dwm3000_usb_dongle/dwm3000_usb_dongle.kicad_sch (KiCad schematic)
At the start: 22 parts, among them J1 USB-4AM103AS, J2 3221-10-0300-00, U1 STM32C071F8P6, U2 XC6220B331MR-G

Commit message: Add USB ESD protection, VBUS fuse/filtering, and power-indicator LED
Cross-checked against an independently-drawn reference schematic and
added the three subsystems it had that this project didn't:

- U3 (USBLC6-2SC6): dual-line USB D+/D- ESD protection, in series
  between the connector and the existing R1/R2 series resistors.
- F1 (500mA PTC fuse) + C4/C8 (100nF HF bypass caps): VBUS now passes
  through a fuse before becoming the board's +5V rail, with extra HF
  bypass at the connector and at the LDO input alongside the existing
  bulk caps.
- D5/R9: an always-on power-indicator LED across +3V3/GND, independent
  of the MCU (unlike the existing D1/D4 status LEDs).

All new chip R/C/LED parts use 0603 (1608 metric) footprints, matching
the rest of the design.

Fixed a bug found along the way: wire_to_power() was called with
"VBUS_RAW" as if it were a power-symbol net (like GND/+3V3/+5V), but
it's just a plain net label -- this referenced a nonexistent
power:VBUS_RAW symbol and crashed kicad-cli's parser. Also fixed U3's
pin routing: its 4 signal pins are only 2.54mm apart, so straight
same-length stubs produced overlapping labels; added a small
jog_label() helper to route each pin out with a short vertical jog
before the label.
Parts:
- added C4, C8: 100nF, Capacitor_SMD:C_0603_1608Metric, symbol Device:C
- added D5: LED, LED_SMD:LED_0603_1608Metric, symbol Device:LED
- added F1: 500mA, Fuse:Fuse_0603_1608Metric, symbol Device:Fuse
- added R9: 1k, Resistor_SMD:R_0603_1608Metric, symbol Device:R
- added U3: USBLC6-2SC6, Package_TO_SOT_SMD:SOT-23-6, symbol Power_Protection:USBLC6-2SC6
Connections:
- net +3V3: now also R9.1
- net +5V: now also C8.1, F1.2, U3.5 (VBUS); no longer J1.1 (VBUS)
- net GND: now also C4.2, C8.2, D5.1 (K), U3.2 (GND)
- net USB_DM: now also U3.6 (I/O1); no longer J1.2 (D-)
- net USB_DP: now also U3.4 (I/O2); no longer J1.3 (D+)
- new net: D5.2 (A), R9.2
- new net USB_DM_RAW: J1.2 (D-), U3.1 (I/O1)
- new net USB_DP_RAW: J1.3 (D+), U3.3 (I/O2)
- new net VBUS_RAW: C4.1, F1.1, J1.1 (VBUS)
